Commit message: 一時的なコミット

File: src/mypkg/urdf/two_link_manipulator_control.urdf.xacro (robot description, xacro)
@@ -7,18 +7,14 @@
         </hardware>
         <joint name="joint1">
-            <command_interface name="position">
-                <param name="min">-3.14</param>
-                <param name="max">3.14</param>
-            </command_interface>
+            <command_interface name="position"/>
             <state_interface name="position"/>
             <state_interface name="velocity"/>
+            <state_interface name="effort"/>
         </joint>
         <joint name="joint2">
-            <command_interface name="position">
-                <param name="min">-3.14</param>
-                <param name="max">3.14</param>
-            </command_interface>
+            <command_interface name="position"/>
             <state_interface name="position"/>
             <state_interface name="velocity"/>
+            <state_interface name="effort"/>
         </joint>
     </ros2_control>
@@ -26,6 +22,6 @@
     <gazebo>
         <plugin name="gazebo_ros2_control" filename="libgazebo_ros2_control.so">
-            <!-- <parameters>$(find mypkg)/config/joint_controllers.yaml</parameters> -->
-            <parameters>$(find mypkg)/config/trajectory_controllers.yaml</parameters>
+            <parameters>$(find mypkg)/config/joint_position_controllers.yaml</parameters>
+            <controlPeriod>0.001</controlPeriod>
         </plugin>
     </gazebo>

File: src/mypkg/urdf/two_link_manipulator_mech.urdf.xacro (robot description, xacro)
@@ -52,5 +52,7 @@
             <mass value="1.0"/>
             <origin xyz="0.25 0 0" rpy="0 0 0"/>
-            <inertia ixx="0.01" ixy="0" ixz="0" iyy="0.01" iyz="0" izz="0.01"/>
+            <inertia ixx="0.0841" ixy="0" ixz="0"
+                     iyy="0.0841" iyz="0"
+                     izz="0.0041"/>
         </inertial>
     </link>
@@ -78,5 +80,7 @@
             <mass value="1.0"/>
             <origin xyz="0.1 0 0" rpy="0 0 0"/>
-            <inertia ixx="0.01" ixy="0" ixz="0" iyy="0.01" iyz="0" izz="0.01"/>
+            <inertia ixx="0.0841" ixy="0" ixz="0"
+                     iyy="0.0841" iyz="0"
+                     izz="0.0041"/>
         </inertial>
     </link>
@@ -90,5 +94,5 @@
         <origin xyz="0 0 0.15" rpy="0 0 0"/>
         <axis xyz="0 0 1"/>
-        <limit lower="-3.14" upper="3.14" effort="100" velocity="1.0"/>
+        <limit lower="-3.14" upper="3.14" effort="100" velocity="100.0"/>
         <dynamics damping="0.7" friction="0.5"/>
     </joint>
@@ -99,6 +103,37 @@
         <origin xyz="0.5 0 0.09" rpy="0 0 0"/>
         <axis xyz="0 0 1"/>
-        <limit lower="-3.14" upper="3.14" effort="100" velocity="1.0"/>
+        <limit lower="-3.14" upper="3.14" effort="100" velocity="100.0"/>
         <dynamics damping="0.7" friction="0.5"/>
     </joint>
+    <!-- ジョイント1のtransmission -->
+    <transmission name="joint1_trans">
+        <type>transmission_interface/SimpleTransmission</type>
+        <joint name="joint1">
+            <!-- <hardwareInterface>hardware_interface/PositionJointInterface</hardwareInterface> -->
+            <hardwareInterface>hardware_interface/EffortJointInterface</hardwareInterface>
+        </joint>
+        <actuator name="joint1_motor">
+            <mechanicalReduction>1</mechanicalReduction>
+        </actuator>
+    </transmission>
+    <!-- ジョイント2のtransmission -->
+    <transmission name="joint2_trans">
+        <type>transmission_interface/SimpleTransmission</type>
+        <joint name="joint2">
+            <!-- <hardwareInterface>hardware_interface/PositionJointInterface</hardwareInterface> -->
+            <hardwareInterface>hardware_interface/EffortJointInterface</hardwareInterface>
+        </joint>
+        <actuator name="joint2_motor">
+            <mechanicalReduction>1</mechanicalReduction>
+        </actuator>
+    </transmission>
+    <!-- Gazeboの物理設定を追加 -->
+    <gazebo reference="joint1">
+        <implicitSpringDamper>true</implicitSpringDamper>
+        <provideFeedback>true</provideFeedback>
+    </gazebo>
+    <gazebo reference="joint2">
+        <implicitSpringDamper>true</implicitSpringDamper>
+        <provideFeedback>true</provideFeedback>
+    </gazebo>
 </robot>
